File: shiftRegBoard/shiftReg.brd (EAGLE design)
At the start: 50.8 x 50.8 mm, 19 parts, among them IC1 SN74HC595N

Commit message: forgot to update
updates of multiple homeworks and sketches
Parts:
- C1: value (none) -> 100u
Changed lines of the file:
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@@
 </autorouter>
 <elements>
-<element name="C1" library="rcl" library_urn="urn:adsk.eagle:library:334" package="C0805" package3d_urn="urn:adsk.eagle:package:23617/2" value="" x="29.21" y="16.51" smashed="yes" rot="R180">
+<element name="C1" library="rcl" library_urn="urn:adsk.eagle:library:334" package="C0805" package3d_urn="urn:adsk.eagle:package:23617/2" value="100u" x="29.21" y="16.51" smashed="yes" rot="R180">
 <attribute name="NAME" x="30.48" y="15.24" size="1.27" layer="25" rot="R180"/>
 <attribute name="POPULARITY" value="63" x="13.97" y="57.15" size="1.778" layer="27" rot="R180" display="off"/>
